File: MCU.kicad_sch (KiCad schematic)
At the start: 64 parts, among them J1 TYPE-C_16PIN_2MD(073), J2 Header-2_54_1x3, SW1 TS-1187A-B-A-B, SW2 TS-1187A-B-A-B, U1 LM3940IMP-3_3/NOPB, U2 RP2040, U3 128Mbit, U4 SN74LV1T34DBVR, Y1 ABM8-272-T3_C20625731

Commit message: pcb finished + production files
Parts:
- C17: LCSC C52923 -> (none)
- R17, R19: now fitted
- U2: Comment (none) -> RP2040; Designator (none) -> U2; JLCPCB Part # (none) -> C2040
