File: numpad.kicad_pcb (KiCad board)
At the start: 2 copper layers, 90 x 132.2 mm, 163 parts, among them J1 TYPE-C_16PIN_2MD(073), J2 Header-2_54_1x3, SW1 TS-1187A-B-A-B, SW2 TS-1187A-B-A-B, U1 LM3940IMP-3_3/NOPB, U2 RP2040, U3 128Mbit, U4 SN74LV1T34DBVR, Y1 ABM8-272-T3_C20625731

Commit message: pcb finished + production files
Parts:
- LED1: renamed from USER RGB
- turned R1 to -90 degrees
- renumbered PWR to LED2, USER to LED3
Routing:
- net +3V3: track 221.6 -> 205.4 mm, vias 15 -> 14
- net /MCU/+3V3_A: track 7.49 -> 8.10 mm
- net ENC2_A: track 41.1 -> 41.7 mm
- added copper zone on B.Cu, net +3V3
